Commit message: nice trajectories. need  to adjust the input and state limits for the joint position.

File: upright_assets/ur5e/collision_links.urdf.xacro (robot description, xacro)
@@ -67,4 +67,32 @@
     <child link="tray_collision_link_3"/>
   </joint>
+   <!-- Wood tray -->
+  <xacro:collision_link name="tray_collision_link_4">
+    <origin rpy="0 0 0" xyz="-0.1 0.1 0.0"/>
+    <geometry>
+      <!-- <sphere radius="0.21"/> -->
+      <sphere radius="0.025"/>
+    </geometry>
+  </xacro:collision_link>
+  <joint name="balanced_object_collision_joint_4" type="fixed">
+    <origin rpy="0 0 0" xyz="0 0 0.0"/>
+    <!-- <origin rpy="0 0 0" xyz="0 0 0"/> -->
+    <parent link="tray"/>
+    <child link="tray_collision_link_4"/>
+  </joint>
+  <!-- Wood tray -->
+  <xacro:collision_link name="tray_collision_link_5">
+    <origin rpy="0 0 0" xyz="-0.1 -0.1 0.0"/>
+    <geometry>
+      <!-- <sphere radius="0.21"/> -->
+      <sphere radius="0.025"/>
+    </geometry>
+  </xacro:collision_link>
+  <joint name="balanced_object_collision_joint_5" type="fixed">
+    <origin rpy="0 0 0" xyz="0 0 0.0"/>
+    <!-- <origin rpy="0 0 0" xyz="0 0 0"/> -->
+    <parent link="tray"/>
+    <child link="tray_collision_link_5"/>
+  </joint>
  <!-- Collision sphere for the base -->
   <xacro:collision_link name="base_collision_link">
@@ -72,5 +100,5 @@
     <geometry>
       <!-- <box size="1.0 0.8 0.3"/> -->
-      <sphere radius="0.2"/>
+      <sphere radius="0.125"/>
     </geometry>
   </xacro:collision_link>

File: upright_assets/ur5e/ur5eTray.urdf (robot description, URDF)
Before this commit: robot robot, 17 links, 16 joints
Links:
- added link tray_collision_link_4; collision sphere radius=0.025; visual sphere radius=0.025
- added link tray_collision_link_5; collision sphere radius=0.025; visual sphere radius=0.025
- link base_collision_link: geometry collision sphere radius=0.125; visual sphere radius=0.125
Joints:
- added joint balanced_object_collision_joint_4: type fixed, parent tray, child tray_collision_link_4, origin xyz=0 0 0.0 rpy=0 0 0
- added joint balanced_object_collision_joint_5: type fixed, parent tray, child tray_collision_link_5, origin xyz=0 0 0.0 rpy=0 0 0

Commit message: Evaluation using a set of custom trajectories -- good with  3s horizon  (slow) -- Object dropped in real (premature stop, non-horizontal tray)/

File: upright_assets/ur5e/collision_links.urdf.xacro (robot description, xacro)
@@ -96,17 +96,30 @@
   </joint>
  <!-- Collision sphere for the base -->
-  <xacro:collision_link name="base_collision_link">
+  <xacro:collision_link name="base_collision_link1">
     <origin rpy="0 0 0" xyz="0 0 0"/>
     <geometry>
       <!-- <box size="1.0 0.8 0.3"/> -->
-      <sphere radius="0.125"/>
-    </geometry>
-  </xacro:collision_link>
-  <!-- TODO it would probably be better to make this relative to the chassis link, so that it includes the calibrated base transform, but this would require some testing as well -->
-  <joint name="base_collision_joint" type="fixed">
+      <sphere radius="0.15"/>
+    </geometry>
+  </xacro:collision_link>
+  <joint name="base_collision_joint1" type="fixed">
     <!-- <origin rpy="0 0 0" xyz="0 0 0.16"/> -->
     <origin rpy="0 0 0" xyz="0 0 0"/>
     <parent link="base_link"/>
-    <child link="base_collision_link"/>
+    <child link="base_collision_link1"/>
+  </joint>
+  <!-- Collision sphere for the base -->
+  <xacro:collision_link name="base_collision_link2">
+    <origin rpy="0 0 0" xyz="0 0 0"/>
+    <geometry>
+      <!-- <box size="1.0 0.8 0.3"/> -->
+      <sphere radius="0.15"/>
+    </geometry>
+  </xacro:collision_link>
+  <joint name="base_collision_joint2" type="fixed">
+    <!-- <origin rpy="0 0 0" xyz="0 0 0.16"/> -->
+    <origin rpy="0 0 0" xyz="0 0 -0.3"/>
+    <parent link="base_link"/>
+    <child link="base_collision_link2"/>
   </joint>
   <!-- Collision sphere for the wrist -->
@@ -158,3 +171,113 @@
     <child link="wrist1_collision_link_4"/>
   </joint>
+<xacro:property name="ground_collision_radius" value="0.2"/>
+<xacro:property name="ground_collision_height" value="-0.5"/>
+<!-- Collision sphere for the base -->
+<xacro:collision_link name="ground_collision_link1">
+  <origin rpy="0 0 0" xyz="0 0 0"/>
+  <geometry>
+    <sphere radius="${ground_collision_radius}"/>
+  </geometry>
+</xacro:collision_link>
+<joint name="ground_collision_link1" type="fixed">
+  <origin rpy="0 0 0" xyz="0 0 ${ground_collision_height}"/>
+  <parent link="base_link"/>
+  <child link="ground_collision_link1"/>
+</joint>
+<!-- Collision sphere for the base -->
+<xacro:collision_link name="ground_collision_link2">
+  <origin rpy="0 0 0" xyz="0 0 0"/>
+  <geometry>
+    <sphere radius="${ground_collision_radius}"/>
+  </geometry>
+</xacro:collision_link>
+<joint name="ground_collision_link2" type="fixed">
+  <origin rpy="0 0 0" xyz="0 ${2 * ground_collision_radius} ${ground_collision_height}"/>
+  <parent link="base_link"/>
+  <child link="ground_collision_link2"/>
+</joint>
+<!-- Collision sphere for the base -->
+<xacro:collision_link name="ground_collision_link3">
+  <origin rpy="0 0 0" xyz="0 0 0"/>
+  <geometry>
+    <sphere radius="${ground_collision_radius}"/>
+  </geometry>
+</xacro:collision_link>
+<joint name="ground_collision_link3" type="fixed">
+  <origin rpy="0 0 0" xyz="0 ${-2 * ground_collision_radius} ${ground_collision_height}"/>
+  <parent link="base_link"/>
+  <child link="ground_collision_link3"/>
+</joint>
+<!-- Collision sphere for the base -->
+<xacro:collision_link name="ground_collision_link4">
+  <origin rpy="0 0 0" xyz="0 0 0"/>
+  <geometry>
+    <sphere radius="${ground_collision_radius}"/>
+  </geometry>
+</xacro:collision_link>
+<joint name="ground_collision_link4" type="fixed">
+  <origin rpy="0 0 0" xyz="${2 * ground_collision_radius} 0 ${ground_collision_height}"/>
+  <parent link="base_link"/>
+  <child link="ground_collision_link4"/>
+</joint>
+<!-- Collision sphere for the base -->
+<xacro:collision_link name="ground_collision_link5">
+  <origin rpy="0 0 0" xyz="0 0 0"/>
+  <geometry>
+    <sphere radius="${ground_collision_radius}"/>
+  </geometry>
+</xacro:collision_link>
+<joint name="ground_collision_link5" type="fixed">
+  <origin rpy="0 0 0" xyz="${4 * ground_collision_radius} 0 ${ground_collision_height}"/>
+  <parent link="base_link"/>
+  <child link="ground_collision_link5"/>
+</joint>
+<!-- Collision sphere for the base -->
+<xacro:collision_link name="ground_collision_link6">
+  <origin rpy="0 0 0" xyz="0 0 0"/>
+  <geometry>
+    <sphere radius="${ground_collision_radius}"/>
+  </geometry>
+</xacro:collision_link>
+<joint name="ground_collision_link6" type="fixed">
+  <origin rpy="0 0 0" xyz="${4 * ground_collision_radius} ${2 * ground_collision_radius} ${ground_collision_height}"/>
+  <parent link="base_link"/>
+  <child link="ground_collision_link6"/>
+</joint>
+<!-- Collision sphere for the base -->
+<xacro:collision_link name="ground_collision_link7">
+  <origin rpy="0 0 0" xyz="0 0 0"/>
+  <geometry>
+    <sphere radius="${ground_collision_radius}"/>
+  </geometry>
+</xacro:collision_link>
+<joint name="ground_collision_link7" type="fixed">
+  <origin rpy="0 0 0" xyz="${4 * ground_collision_radius} ${-2 * ground_collision_radius} ${ground_collision_height}"/>
+  <parent link="base_link"/>
+  <child link="ground_collision_link7"/>
+</joint>
+<!-- Collision sphere for the base -->
+<xacro:collision_link name="ground_collision_link8">
+  <origin rpy="0 0 0" xyz="0 0 0"/>
+  <geometry>
+    <sphere radius="${ground_collision_radius}"/>
+  </geometry>
+</xacro:collision_link>
+<joint name="ground_collision_link8" type="fixed">
+  <origin rpy="0 0 0" xyz="${2 * ground_collision_radius} ${-2 * ground_collision_radius} ${ground_collision_height}"/>
+  <parent link="base_link"/>
+  <child link="ground_collision_link8"/>
+</joint>
+<!-- Collision sphere for the base -->
+<xacro:collision_link name="ground_collision_link9">
+  <origin rpy="0 0 0" xyz="0 0 0"/>
+  <geometry>
+    <sphere radius="${ground_collision_radius}"/>
+  </geometry>
+</xacro:collision_link>
+<joint name="ground_collision_link9" type="fixed">
+  <origin rpy="0 0 0" xyz="${2 * ground_collision_radius} ${2 * ground_collision_radius} ${ground_collision_height}"/>
+  <parent link="base_link"/>
+  <child link="ground_collision_link9"/>
+</joint>
 </robot>

File: upright_assets/ur5e/ur5eTray.urdf (robot description, URDF)
Before this commit: robot robot, 19 links, 18 joints
Links:
- removed link base_collision_link
- added link base_collision_link1; collision sphere radius=0.15; visual sphere radius=0.15
- added link base_collision_link2; collision sphere radius=0.15; visual sphere radius=0.15
- added link ground_collision_link1; collision sphere radius=0.2; visual sphere radius=0.2
- added link ground_collision_link2; collision sphere radius=0.2; visual sphere radius=0.2
- added link ground_collision_link3; collision sphere radius=0.2; visual sphere radius=0.2
- added link ground_collision_link4; collision sphere radius=0.2; visual sphere radius=0.2
- added link ground_collision_link5; collision sphere radius=0.2; visual sphere radius=0.2
- added link ground_collision_link6; collision sphere radius=0.2; visual sphere radius=0.2
- added link ground_collision_link7; collision sphere radius=0.2; visual sphere radius=0.2
- added link ground_collision_link8; collision sphere radius=0.2; visual sphere radius=0.2
- added link ground_collision_link9; collision sphere radius=0.2; visual sphere radius=0.2
Joints:
- removed joint base_collision_joint
- added joint base_collision_joint1: type fixed, parent base_link, child base_collision_link1, origin xyz=0 0 0 rpy=0 0 0
- added joint base_collision_joint2: type fixed, parent base_link, child base_collision_link2, origin xyz=0 0 -0.3 rpy=0 0 0
- added joint ground_collision_link1: type fixed, parent base_link, child ground_collision_link1, origin xyz=0 0 -0.5 rpy=0 0 0
- added joint ground_collision_link2: type fixed, parent base_link, child ground_collision_link2, origin xyz=0 0.4 -0.5 rpy=0 0 0
- added joint ground_collision_link3: type fixed, parent base_link, child ground_collision_link3, origin xyz=0 -0.4 -0.5 rpy=0 0 0
- added joint ground_collision_link4: type fixed, parent base_link, child ground_collision_link4, origin xyz=0.4 0 -0.5 rpy=0 0 0
- added joint ground_collision_link5: type fixed, parent base_link, child ground_collision_link5, origin xyz=0.8 0 -0.5 rpy=0 0 0
- added joint ground_collision_link6: type fixed, parent base_link, child ground_collision_link6, origin xyz=0.8 0.4 -0.5 rpy=0 0 0
- added joint ground_collision_link7: type fixed, parent base_link, child ground_collision_link7, origin xyz=0.8 -0.4 -0.5 rpy=0 0 0
- added joint ground_collision_link8: type fixed, parent base_link, child ground_collision_link8, origin xyz=0.4 -0.4 -0.5 rpy=0 0 0
- added joint ground_collision_link9: type fixed, parent base_link, child ground_collision_link9, origin xyz=0.4 0.4 -0.5 rpy=0 0 0
